File: snus_tomogatchi.kicad_sch (KiCad schematic)
At the start: 27 parts, among them J2 Conn_01x04, J3 USB_B_Micro, SW1 SW_Push, SW2 SW_Push, SW3 SW_DPDT_x2, U1 ESP32-C3FH4, U3 LD1117S33TR_SOT223, Y1 ABM11W-40.0000MHZ-6-B1U-T3

Commit message: Add files via upload
Parts:
- removed SW3: SW_DPDT_x2, symbol Switch:SW_DPDT_x2
- added S1: SSAJ120100, SamacSys_Parts:SSAJ120100, symbol SamacSys_Parts:SSAJ120100
- BT1, BT2: footprint (none) -> SamacSys_Parts:BATHLD007SMTTR
- C1, C10, C11, C12, C2, C3, C4, C5, C6, C7, C8, C9: footprint (none) -> Capacitor_SMD:C_0603_1608Metric_Pad1.08x0.95mm_HandSolder
- J2: footprint (none) -> Connector_PinHeader_2.54mm:PinHeader_1x04_P2.54mm_Vertical
- R1, R2, R3: footprint (none) -> Resistor_SMD:R_0603_1608Metric_Pad0.98x0.95mm_HandSolder
- SW1, SW2: footprint (none) -> Button_Switch_THT:SW_Tactile_SKHH_Angled
Connections:
- net +3V3: now also C12.1, U3.2 (VO)
- net +5V: now also S1.5 (MP2)
- net 6V: now also S1.4 (MP1)
- net V_IN: now reaches C11.1, U3.3 (VI)
- net V_IN: now also S1.3 (COM)
- no-connect marks 17 -> 18
Other:
- moved on the sheet: C11, C12, U3
